File: pcb design/Steno Keyboard.kicad_pcb (KiCad board)
At the start: 2 copper layers, 259.2 x 79.2 mm, 64 parts, among them SW1 SW_DIP_x01, SW10 SW_DIP_x01, SW11 SW_DIP_x01, SW12 SW_DIP_x01, SW13 SW_DIP_x01, SW14 SW_DIP_x01, SW15 SW_DIP_x01, SW16 SW_DIP_x01, SW17 SW_DIP_x01, SW18 SW_DIP_x01, SW19 SW_DIP_x01, SW2 SW_DIP_x01, SW20 SW_DIP_x01, SW21 SW_DIP_x01, SW22 SW_DIP_x01, SW23 SW_DIP_x01, SW24 SW_DIP_x01, SW25 SW_DIP_x01, SW26 SW_DIP_x01, SW27 SW_DIP_x01, SW28 SW_DIP_x01, SW3 SW_DIP_x01, SW4 SW_DIP_x01, SW5 SW_DIP_x01, SW6 SW_DIP_x01, SW7 SW_DIP_x01, SW8 SW_DIP_x01, SW9 SW_DIP_x01

Commit message: updated PCB design
Parts:
- added G***: LOGO, LOGO, F.Cu at (39.5, 87.0)
- added G***: LOGO, LOGO, F.Cu at (137.5, 77.5)
- added G***: LOGO, LOGO, F.Cu at (246.0, 87.5)
- added R1: 0, Resistor_SMD:R_1206_3216Metric_Pad1.30x1.75mm_HandSolder, B.Cu at (41.5, 55.0)
- added R10: 0, Resistor_SMD:R_1206_3216Metric_Pad1.30x1.75mm_HandSolder, B.Cu at (194.5, 55.0)
- added R11: 0, Resistor_SMD:R_1206_3216Metric_Pad1.30x1.75mm_HandSolder, B.Cu at (214.5, 55.0)
- added R12: 0, Resistor_SMD:R_1206_3216Metric_Pad1.30x1.75mm_HandSolder, B.Cu at (234.5, 55.0)
- added R13: 0, Resistor_SMD:R_1206_3216Metric_Pad1.30x1.75mm_HandSolder, B.Cu at (254.5, 55.0)
- added R15: 0, Resistor_SMD:R_1206_3216Metric_Pad1.30x1.75mm_HandSolder, B.Cu at (174.5, 75.0)
- added R16: 0, Resistor_SMD:R_1206_3216Metric_Pad1.30x1.75mm_HandSolder, B.Cu at (194.5, 75.0)
- added R17: 0, Resistor_SMD:R_1206_3216Metric_Pad1.30x1.75mm_HandSolder, B.Cu at (121.8, 55.0)
- added R18: 0, Resistor_SMD:R_1206_3216Metric_Pad1.30x1.75mm_HandSolder, B.Cu at (121.8, 75.0)
- added R19: 0, Resistor_SMD:R_1206_3216Metric_Pad1.30x1.75mm_HandSolder, B.Cu at (214.5, 75.0)
- added R2: 0, Resistor_SMD:R_1206_3216Metric_Pad1.30x1.75mm_HandSolder, B.Cu at (61.5, 55.0)
- added R3: 0, Resistor_SMD:R_1206_3216Metric_Pad1.30x1.75mm_HandSolder, B.Cu at (81.8, 55.0)
- added R4: 0, Resistor_SMD:R_1206_3216Metric_Pad1.30x1.75mm_HandSolder, B.Cu at (101.8, 55.0)
- added R6: 0, Resistor_SMD:R_1206_3216Metric_Pad1.30x1.75mm_HandSolder, B.Cu at (81.5, 75.0)
- added R7: 0, Resistor_SMD:R_1206_3216Metric_Pad1.30x1.75mm_HandSolder, B.Cu at (101.5, 75.0)
- added R9: 0, Resistor_SMD:R_1206_3216Metric_Pad1.30x1.75mm_HandSolder, B.Cu at (174.5, 55.0)
- D1, D10, D11, D12, D13, D14, D15, D16, D17, D18, D19, D2, D20, D21, D22, D23, D24, D25, D26, D27, D28, D3, D4, D5, D6, D7, D8, D9: footprint Diode_THT:D_DO-35_SOD27_P7.62mm_Horizontal -> Diode_SMD:D_SOD-123
- moved D14 2.00 mm to (159.0, 53.3)
- moved D15 2.00 mm to (179.0, 53.3)
- moved D16 2.00 mm to (199.0, 53.3)
- moved D17 2.00 mm to (219.0, 53.3)
- moved D18 2.00 mm to (239.0, 53.3)
- moved D20 2.00 mm to (159.0, 73.3)
- moved D21 2.00 mm to (179.0, 73.3)
- moved D22 2.00 mm to (199.0, 73.3)
- moved D23 2.00 mm to (219.0, 73.3)
- moved D24 2.00 mm to (239.0, 73.3)
- moved D26 2.00 mm to (159.0, 93.3)
- moved D27 2.00 mm to (179.0, 93.3)
- moved D28 2.00 mm to (199.0, 93.3)
- moved D19 2.00 mm to (259.0, 53.3)
- moved D25 2.00 mm to (259.0, 73.3)
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Connections:
- D1 pad 1: Row 0 -> Net-(D1-K)
- D10 pad 1: Row 1 -> Net-(D10-K)
- D15 pad 1: Row 3 -> Net-(D15-K)
- D16 pad 1: Row 3 -> Net-(D16-K)
- D17 pad 1: Row 3 -> Net-(D17-K)
- D18 pad 1: Row 3 -> Net-(D18-K)
- D19 pad 1: Row 3 -> Net-(D19-K)
- D2 pad 1: Row 0 -> Net-(D2-K)
- D21 pad 1: Row 4 -> Net-(D21-K)
- D22 pad 1: Row 4 -> Net-(D22-K)
- D23 pad 1: Row 4 -> Net-(D23-K)
- D24 pad 1: Row 4 -> Net-(D23-K)
- D25 pad 1: Row 4 -> Net-(D23-K)
- D3 pad 1: Row 0 -> Net-(D3-K)
- D4 pad 1: Row 0 -> Net-(D4-K)
- D5 pad 1: Row 0 -> Net-(D5-K)
- D6 pad 1: Row 1 -> Net-(D6-K)
- D7 pad 1: Row 1 -> Net-(D6-K)
- D8 pad 1: Row 1 -> Net-(D6-K)
- D9 pad 1: Row 1 -> Net-(D9-K)
Routing:
- net Row 0: track 120.3 -> 22.3 mm
- net Row 1: track 132.3 -> 38.7 mm
- net Row 3: track 121.8 -> 40.5 mm
- net Row 4: track 141.9 -> 63.5 mm
- net Net-(D6-K): track 0.00 -> 54.0 mm
- net Net-(D23-K): track 0.00 -> 43.0 mm
- net Net-(D3-K): track 0.00 -> 17.2 mm
- net Net-(D10-K): track 0.00 -> 17.2 mm
- net Net-(D2-K): track 0.00 -> 16.9 mm
- net Net-(D21-K): track 0.00 -> 16.9 mm
- net Net-(D4-K): track 0.00 -> 16.9 mm
- net Net-(D18-K): track 0.00 -> 16.9 mm
- net Net-(D22-K): track 0.00 -> 16.9 mm
- net Net-(D17-K): track 0.00 -> 16.9 mm
- net Net-(D16-K): track 0.00 -> 16.9 mm
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Other:
- board text added: "NEBC PROJECT #2"
