File: pcb design/Steno Keyboard.kicad_sch (KiCad schematic)
At the start: 57 parts, among them SW1 SW_DIP_x01, SW10 SW_DIP_x01, SW11 SW_DIP_x01, SW12 SW_DIP_x01, SW13 SW_DIP_x01, SW14 SW_DIP_x01, SW15 SW_DIP_x01, SW16 SW_DIP_x01, SW17 SW_DIP_x01, SW18 SW_DIP_x01, SW19 SW_DIP_x01, SW2 SW_DIP_x01, SW20 SW_DIP_x01, SW21 SW_DIP_x01, SW22 SW_DIP_x01, SW23 SW_DIP_x01, SW24 SW_DIP_x01, SW25 SW_DIP_x01, SW26 SW_DIP_x01, SW27 SW_DIP_x01, SW28 SW_DIP_x01, SW3 SW_DIP_x01, SW4 SW_DIP_x01, SW5 SW_DIP_x01, SW6 SW_DIP_x01, SW7 SW_DIP_x01, SW8 SW_DIP_x01, SW9 SW_DIP_x01

Commit message: updated PCB design
Parts:
- added R1, R10, R11, R12, R13, R15, R16, R17, R18, R19, R2, R3, R4, R6, R7, R9: 0, Resistor_SMD:R_1206_3216Metric_Pad1.30x1.75mm_HandSolder, symbol ScottoKeebs:Placeholder_Resistor
- D1, D10, D11, D12, D13, D14, D15, D16, D17, D18, D19, D2, D20, D21, D22, D23, D24, D25, D26, D27, D28, D3, D4, D5, D6, D7, D8, D9: footprint Diode_THT:D_DO-35_SOD27_P7.62mm_Horizontal -> Diode_SMD:D_SOD-123
Connections:
- net Row 0: now also R17.2; no longer D1.1 (K), D2.1 (K), D3.1 (K), D4.1 (K), D5.1 (K)
- net Row 1: now also R18.2; no longer D10.1 (K), D6.1 (K), D7.1 (K), D8.1 (K), D9.1 (K)
- net Row 3: now also R9.1; no longer D15.1 (K), D16.1 (K), D17.1 (K), D18.1 (K), D19.1 (K)
- net Row 4: now also R15.1; no longer D21.1 (K), D22.1 (K), D23.1 (K), D24.1 (K), D25.1 (K)
- new net: D9.1 (K), R6.2, R7.1
- new net: D10.1 (K), R18.1, R7.2
- new net: D17.1 (K), R11.2, R12.1
- new net: D6.1 (K), D7.1 (K), D8.1 (K), R6.1
- new net: D1.1 (K), R1.1
- new net: D2.1 (K), R1.2, R2.1
- new net: D4.1 (K), R3.2, R4.1
- new net: D3.1 (K), R2.2, R3.1
- new net: D15.1 (K), R10.1, R9.2
- new net: D5.1 (K), R17.1, R4.2
- new net: D21.1 (K), R15.2, R16.1
- new net: D23.1 (K), D24.1 (K), D25.1 (K), R19.2
- new net: D16.1 (K), R10.2, R11.1
- new net: D18.1 (K), R12.2, R13.1
- new net: D19.1 (K), R13.2
- new net: D22.1 (K), R16.2, R19.1
Other:
- moved on the sheet: D1, D10, D11, D12, D13, D14, D15, D16, D17, D18, D19, D2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
